Commit message: Fix URDF mesh paths, update model.sdf and setup.py

File: src/ika_parkur/urdf/arac.urdf (robot description, URDF)
Before this commit: robot teknofest_ika, 6 links, 5 joints
Links:
- link base_link: geometry collision box size=1.0 0.5 0.3; visual mesh filename=file:///home/bugra16/ika_ws/src/teknofest_ika/src/ika_parku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 scale=0.001 0.001 0.001
- link sag_arka_teker: geometry collision cylinder length=0.15 radius=0.18; visual mesh filename=file:///home/bugra16/ika_ws/src/teknofest_ika/src/ika_parku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 scale=0.001 0.001 0.001
- link sag_on_teker: geometry collision cylinder length=0.15 radius=0.18; visual mesh filename=file:///home/bugra16/ika_ws/src/teknofest_ika/src/ika_parku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 scale=0.001 0.001 0.001
- link sol_arka_teker: geometry collision cylinder length=0.15 radius=0.18; visual mesh filename=file:///home/bugra16/ika_ws/src/teknofest_ika/src/ika_parku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 scale=0.001 0.001 0.001
- link sol_on_teker: geometry collision cylinder length=0.15 radius=0.18; visual mesh filename=file:///home/bugra16/ika_ws/src/teknofest_ika/src/ika_parku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 scale=0.001 0.001 0.001
