Commit message: refactor: paket yapısı src/ika_parkur/ altından köke taşındı

File: urdf/arac.urdf (robot description, URDF)
Before this commit: robot teknofest_ika, 6 links, 5 joints
Links:
- added link imu_link, mass 0.01
- added link kamera_link, mass 0.1; visual box size=0.05 0.05 0.05
- added link lidar_link, mass 0.1; visual cylinder length=0.05 radius=0.05
- link base_link: geometry collision box size=1.0 0.5 0.3; visual mesh filename=package://teknofest_ika/meshes/govde.stl scale=0.001 0.001 0.001
- link sag_arka_teker: geometry collision cylinder length=0.15 radius=0.18; visual mesh filename=package://teknofest_ika/meshes/tekerlek.stl scale=0.001 0.001 0.001
- link sag_on_teker: geometry collision cylinder length=0.15 radius=0.18; visual mesh filename=package://teknofest_ika/meshes/tekerlek.stl scale=0.001 0.001 0.001
- link sol_arka_teker: geometry collision cylinder length=0.15 radius=0.18; visual mesh filename=package://teknofest_ika/meshes/tekerlek.stl scale=0.001 0.001 0.001
- link sol_on_teker: geometry collision cylinder length=0.15 radius=0.18; visual mesh filename=package://teknofest_ika/meshes/tekerlek.stl scale=0.001 0.001 0.001
Joints:
- added joint imu_joint: type fixed, parent base_link, child imu_link, origin xyz=0 0 0 rpy=0 0 0
- added joint kamera_joint: type fixed, parent base_link, child kamera_link, origin xyz=0.55 0 0.20 rpy=0 0 0
- added joint lidar_joint: type fixed, parent base_link, child lidar_link, origin xyz=0.0 0 0.30 rpy=0 0 0

Commit message: fix: wheel axis düzeltildi, spin behavior eklendi, Nav2 ilk otonom test başarılı

File: urdf/arac.urdf (robot description, URDF)
Before this commit: robot teknofest_ika, 9 links, 8 joints
Joints:
- joint sag_arka_joint: axis 0 1 0 -> 0 -1 0
- joint sag_on_joint: axis 0 1 0 -> 0 -1 0
- joint sol_arka_joint: axis 0 1 0 -> 0 -1 0
- joint sol_on_joint: axis 0 1 0 -> 0 -1 0

Commit message: feat: performans optimizasyonlari, bug duzeltmeleri ve yeni node'lar
- DetectionsStore.update_field() eklendi: parcali topic guncellemelerinde
  e_stop/manual_mod sifirlanma bug'i duzeltildi
- kayar_engel_kalman: LiDAR scan isleme NumPy ile vektorize edildi (~30x hizli)
- seri_kopru: struct.unpack birlestirildi, _normalize math.remainder ile
  guncellendi, RC mesaji onceden tahsis edildi
- ackermann_converter: AckermannDriveStamped mesajlari onceden tahsis edildi
- Yeni node'lar: e_stop_node, mod_yoneticisi, lora_gcs, kayar_engel_costmap,
  koni_costmap
- Yeni launch: gercek_arac.launch.py (tam yaris stack'i), gercek_harita.launch.py
- Eski/gereksiz dosyalar silindi: slam.launch.py, teknofest_ika/topics.py,
  tabelalar_fixed/yedek.dae
- 58/58 birim testi gecti

File: urdf/arac.urdf (robot description, URDF)
Before this commit: robot teknofest_ika, 9 links, 8 joints
Links:
- added link os30a_link, mass 0.15; visual box size=0.06 0.06 0.04
Joints:
- added joint os30a_joint: type fixed, parent base_link, child os30a_link, origin xyz=0.30 0 0.20 rpy=0 0 0

Commit message: feat: YOLO class_id duzeltmesi, DIK_EGIM waypoint bolunmesi, stop cooldown optimizasyonu
- yolo_adapter_node: class_id sabitleri gercek model siralamasina (alfabetik)
  gore duzeltildi; Tabela_12 bilinmeyen sinif olarak isaretlendi
- terrain_adapter: CLASS_TO_TERRAIN 10->16 giris, tum class_id'ler dogru
  terrain profiliyle eslendi; Tabela_10/DIK_EGIM_CIKIS normal profile alindi
- misyon_fsm: STOP cooldown 6s->3s (rampa cift STOP icin yeterli aralik)
- waypoints.yaml: DIK_EGIM->GIRIS+CIKIS bolundu (§6.10 cikis STOP icin);
  YAN_EGIM_2 kaldirildi (Tabela_10 aslinda DIK_EGIM cikis tabelasi)
- test_birim.py: stop_var ardisik frame, FSM cooldown, hizlanma profili,
  DetectionsStore testleri eklendi (95/95 gecti)
- Yeni node'lar: cone_fusion, lane_detection, preprocessing, servo_controller,
  targeting, yolo_adapter, yolo_detection, watchdog, utils/

File: urdf/arac.urdf (robot description, URDF)
Before this commit: robot teknofest_ika, 10 links, 9 joints
Joints:
- joint sol_arka_joint: origin xyz=-0.60 0.320 -0.10 rpy=0 0 0 -> xyz=-0.60 0.335 -0.10 rpy=0 0 0
- joint sol_on_joint: origin xyz=0.50 0.320 -0.10 rpy=0 0 0 -> xyz=0.50 0.335 -0.10 rpy=0 0 0

Commit message: feat: gercek_arac tam entegrasyon — IMX258, DUBIN planner, class_id duzeltme
- ekf.yaml: yaw odom'dan kapatildi (IMU'dan alinir), imu_remove_gravity false
- nav2_params.yaml: Reeds-Shepp -> DUBIN planner, velocity_smoother eklendi
- nav2_params_test.yaml: lookahead 1.0, max_angular_vel 1.0, costmap 10Hz
- gercek_arac.launch.py: IMX258 v4l2 node eklendi, teknofest_harita.pgm, koni_costmap kaldirildi
- yolo_detection_node.py: CLASS_NAMES 16 sinif, alfabetik model sirasi
- topics.py: SCAN_LIDAR_TOPIC eklendi, YOLO_CLASSES 16 eleman, class_id aciklamalari duzeltildi
- cone_fusion_node.py: PointCloud2 frame_id base_footprint olarak uzerine yazildi
- kayar_engel_costmap.py: varsayilan frame laser -> lidar_link
- preprocessing_node.py + scan_relay.py: topic'ler topics.py sabitlerinden aliniyor
- anti_rollback.py: E-STOP entegrasyonu eklendi
- watchdog.py: /scan -> /scan_lidar, startup grace 15 -> 30s
- urdf/arac.urdf: kamera_link -> camera_link (ROS standart)
- package.xml: vision_msgs, v4l2_camera, smach bagimliliklari eklendi

File: urdf/arac.urdf (robot description, URDF)
Before this commit: robot teknofest_ika, 10 links, 9 joints
Links:
- removed link kamera_link
- added link camera_link, mass 0.1; visual box size=0.05 0.05 0.05
Joints:
- joint kamera_joint: child kamera_link -> camera_link

Commit message: fix: kritik guvenlik ve sartname uyumsuzluklarini giderildi
- max_speed limiti VESC sinirina (3.0 m/s) cekildi
- lazer atis sonrasi hareket kilidinin acilmama hatasi duzeltildi
- nisan kamerasi gercek taret kamerasina baglandi
- e-stop/watchdog ayrilik ilkesi guclendirildi
- dik egim STOP tespiti icin konum tabanli yedek tetikleyici eklendi
- arduino fren mantigi (coast->short-brake) duzeltildi
- YOLO guven esigi ve ardisik-kare dogrulama tutarlilastirildi
- kayar engel yon tespiti hiz bilesenine gore iyilestirildi
- imu hiz sinirinin Nav2'ye anlik iletilmesi saglandi
- yagmur filtresi yanlis pozitif riski azaltildi
- test_birim.py gercek uretim kodunu (pure_logic.py) test edecek sekilde
  yeniden yazildi
- olu simulasyon/test dosyalari ve CI/Makefile yol hatalari temizlendi
- wheelbase ve AMCL config tutarsizliklari giderildi

File: urdf/arac.urdf (robot description, URDF)
Before this commit: robot teknofest_ika, 10 links, 9 joints
Joints:
- joint sag_arka_joint: origin xyz=-0.60 -0.335 -0.10 rpy=0 0 0 -> xyz=-0.275 -0.335 -0.10 rpy=0 0 0
- joint sag_on_joint: origin xyz=0.50 -0.335 -0.10 rpy=0 0 0 -> xyz=0.275 -0.335 -0.10 rpy=0 0 0
- joint sol_arka_joint: origin xyz=-0.60 0.335 -0.10 rpy=0 0 0 -> xyz=-0.275 0.335 -0.10 rpy=0 0 0
- joint sol_on_joint: origin xyz=0.50 0.335 -0.10 rpy=0 0 0 -> xyz=0.275 0.335 -0.10 rpy=0 0 0
