Commit message: fix: LiDAR montaj donusunu ve frame adini TF'e tasi
LiDAR govdeye 93.3 derece donuk monte (sahada huniyle cift yonlu kalibre
edildi). huni_reaktif bu duzeltmeyi kendi icinde ham /scan uzerinde
aci_offset_deg ile yapar ve TF'ten etkilenmez; Nav2 costmap ise YALNIZ TF'e
bakar. Donus verilmediginde tum engeller 93 derece kaydirilarak yerlestirilir
— arac duvari solunda sanip saga kirar.

- lidar_link -> laser_frame: surucunun yayinladigi frame_id ile birebir ayni
  olmali (lydia_ortam/tmini_pro.yaml). Farkli isimde /scan hicbir TF'e
  oturmaz ve costmap bos kalir.
- rpy 0 0 1.6284 (= 93.3 derece), z 0.55 m (zeminden tarama duzlemine olculdu).
  Onceki degerler rpy 0 0 0 ve z 0.30 idi; acilis betigindeki statik yayinci
  ise 0.55 kullaniyordu — uc kaynak birbirini tutmuyordu.

File: urdf/arac.urdf (robot description, URDF)
Before this commit: robot teknofest_ika, 10 links, 9 joints
Links:
- removed link lidar_link
- added link laser_frame, mass 0.1; visual cylinder length=0.05 radius=0.05
Joints:
- joint lidar_joint: child lidar_link -> laser_frame; origin xyz=0.0 0 0.30 rpy=0 0 0 -> xyz=0.0 0 0.55 rpy=0 0 1.6284

Commit message: chore: kullanilmayan varliklari ve kopuk koni koprusunu kaldir
materials/ Gazebo tabela dokulariydi; repoda .world/.sdf yok, simulasyon
hic kurulmadi. meshes/ yalnizca urdf'in <visual> bloklarindan okunuyordu ve
o bloklar collision'daki primitiflerin ayni sekilleri; gorsel geometri box
ve cylinder'a cevrildi, boylece rviz2 araci yine cizer. Tekerleklerde taraf
basina farkli rpy STL yonelimi icindi, silindir simetrik oldugu icin dordu
de ayni.

koni_costmap.py iki ucundan da kopuktu: abone oldugu /cone_positions'a
kimse yayin yapmiyor, urettigi /cone_cloud'u da Nav2 dinlemiyor (costmap
/costmap/cone_cloud bekliyor, onu cone_fusion_node yaziyor).

DFRobot_BMI160'ta kutuphanenin kendi ornekleri silindi, surucu duruyor.

File: urdf/arac.urdf (robot description, URDF)
Before this commit: robot teknofest_ika, 10 links, 9 joints
Links:
- link base_link: geometry collision box size=1.0 0.5 0.3; visual box size=1.0 0.5 0.3
- link sag_arka_teker: geometry collision cylinder length=0.15 radius=0.18; visual cylinder length=0.15 radius=0.18
- link sag_on_teker: geometry collision cylinder length=0.15 radius=0.18; visual cylinder length=0.15 radius=0.18
- link sol_arka_teker: geometry collision cylinder length=0.15 radius=0.18; visual cylinder length=0.15 radius=0.18
- link sol_on_teker: geometry collision cylinder length=0.15 radius=0.18; visual cylinder length=0.15 radius=0.18

Commit message: fix: olculen dingil arasini ve araca ozgu iki duzeltmeyi depoya al
Uc degisiklik de aracin calisma agacinda vardi ama hicbir uzak dalda
karsiligi yoktu; kaynagi 2026-08-20 Jetson taramasi.

wheelbase 0.55 -> 1.40 (2026-07-27 araçtan olculdu). Placeholder deger
dort yerde daha yansiyordu: urdf teker joint'leri (±0.275 -> ±0.70),
ekf.yaml ve nav2_params.yaml basliklari, test_birim.py. Nav2'nin
minimum_turning_radius'u da bu degerden turedigi icin 0.95 -> 2.42
guncellendi; planlayici bu olmadan aracin donemeyecegi viraj ciziyordu.
huni_reaktif'in k_yaw ayari L=0.55 zincirinden gecmisti — dugum arsivde,
reaktif surise donulurse yeniden ayarlanmali.

ackermann_converter'a otomatik_fren parametresi: fren hatti kontrolcunun
gaz kesme girisini de cektigi icin hiz her dustugunde gaz kesiliyor.

yolo_detection_node .engine icin once ultralytics deniyor — `yolo export`
engine'i ultralytics formatinda ve ham TensorRTInferer acamiyor, node
sessizce yavas .pt yoluna dusuyordu. Ayni duzeltme targeting_node'da vardi.

File: urdf/arac.urdf (robot description, URDF)
Before this commit: robot teknofest_ika, 10 links, 9 joints
Joints:
- joint sag_arka_joint: origin xyz=-0.275 -0.335 -0.10 rpy=0 0 0 -> xyz=-0.70 -0.335 -0.10 rpy=0 0 0
- joint sag_on_joint: origin xyz=0.275 -0.335 -0.10 rpy=0 0 0 -> xyz=0.70 -0.335 -0.10 rpy=0 0 0
- joint sol_arka_joint: origin xyz=-0.275 0.335 -0.10 rpy=0 0 0 -> xyz=-0.70 0.335 -0.10 rpy=0 0 0
- joint sol_on_joint: origin xyz=0.275 0.335 -0.10 rpy=0 0 0 -> xyz=0.70 0.335 -0.10 rpy=0 0 0
